File: kicad/neopeto/neopeto.kicad_pcb (KiCad board)
At the start: 2 copper layers, 99.1 x 74.9 mm, 82 parts, among them J1 Conn_01x10_Pin, J2 Conn_01x10_Pin, J3 Conn_01x10_Pin, J4 PJ-307, U1 74HC00, U10 74HC590, U11 74HC590, U12 74HC590, U13 74HC245, U14 K6X4008C1F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

Commit message: wip
Parts:
- added G***: LOGO, LOGO, F.Cu at (85.4, 48.1)
Other:
- board text added: "PÉTOMANE RINGARD"
- board text removed: "PÉTOMANE NOUVEAU"

Commit message: wip
Parts:
- added C22: 100nF, Capacitor_SMD:C_0603_1608Metric, F.Cu at (122.0, 29.6)
- added C23: 10uF, Capacitor_SMD:C_0805_2012Metric, F.Cu at (120.7, 35.3)
- added C24: 1uF, Capacitor_SMD:C_0603_1608Metric, F.Cu at (122.4, 32.8)
- added D1: LED_Small, LED_SMD:LED_0402_1005Metric, F.Cu at (71.0, 26.9)
- added D10: LED_Small, LED_SMD:LED_0402_1005Metric, F.Cu at (88.8, 26.9)
- added D11: LED_Small, LED_SMD:LED_0402_1005Metric, F.Cu at (90.3, 26.9)
- added D12: LED_Small, LED_SMD:LED_0402_1005Metric, F.Cu at (92.3, 26.9)
- added D13: LED_Small, LED_SMD:LED_0402_1005Metric, F.Cu at (94.3, 26.9)
- added D14: LED_Small, LED_SMD:LED_0402_1005Metric, F.Cu at (96.3, 26.9)
- added D15: LED_Small, LED_SMD:LED_0402_1005Metric, F.Cu at (98.3, 26.9)
- added D16: LED_Small, LED_SMD:LED_0402_1005Metric, F.Cu at (100.1, 26.9)
- added D17: LED_Small, LED_SMD:LED_0402_1005Metric, F.Cu at (102.1, 26.9)
- added D18: LED_Small, LED_SMD:LED_0402_1005Metric, F.Cu at (104.1, 26.9)
- added D19: LED_Small, LED_SMD:LED_0402_1005Metric, F.Cu at (106.1, 26.9)
- added D2: LED_Small, LED_SMD:LED_0402_1005Metric, F.Cu at (73.0, 26.9)
- added D20: LED_Small, LED_SMD:LED_0402_1005Metric, F.Cu at (108.1, 26.9)
- added D21: BAT54S, Package_TO_SOT_SMD:SOT-23, F.Cu at (116.9, 33.7)
- added D3: LED_Small, LED_SMD:LED_0402_1005Metric, F.Cu at (75.0, 26.9)
- added D4: LED_Small, LED_SMD:LED_0402_1005Metric, F.Cu at (77.0, 26.9)
- added D5: LED_Small, LED_SMD:LED_0402_1005Metric, F.Cu at (79.0, 26.9)
- added D6: LED_Small, LED_SMD:LED_0402_1005Metric, F.Cu at (80.8, 26.9)
- added D7: LED_Small, LED_SMD:LED_0402_1005Metric, F.Cu at (82.8, 26.9)
- added D8: LED_Small, LED_SMD:LED_0402_1005Metric, F.Cu at (84.8, 26.9)
- added D9: LED_Small, LED_SMD:LED_0402_1005Metric, F.Cu at (86.8, 26.9)
- added JP1: SolderJumper_3_Bridged12, Jumper:SolderJumper-3_P1.3mm_Bridged12_RoundedPad1.0x1.5mm_NumberLabels, F.Cu at (142.1, 60.9)
- added R17: 470, Resistor_SMD:R_0805_2012Metric, F.Cu at (113.1, 32.8)
- added R18: 470, Resistor_SMD:R_0805_2012Metric, F.Cu at (107.7, 30.9)
- added R19: 470, Resistor_SMD:R_0805_2012Metric, F.Cu at (88.2, 30.7)
- added R20: 470, Resistor_SMD:R_0805_2012Metric, F.Cu at (96.4, 30.9)
- added R21: 470, Resistor_SMD:R_0805_2012Metric, F.Cu at (100.9, 30.9)
- added R22: 100K, Resistor_SMD:R_0805_2012Metric, F.Cu at (127.9, 35.1)
- added R23: 100K, Resistor_SMD:R_0805_2012Metric, F.Cu at (123.0, 26.9)
- added R24: 100K, Resistor_SMD:R_0805_2012Metric, F.Cu at (119.9, 28.1)
- added R25: 12K, Resistor_SMD:R_0805_2012Metric, F.Cu at (119.9, 31.9)
- added TP13: TestPoint, TestPoint:TestPoint_Pad_D1.5mm, B.Cu at (111.8, 27.9)
- added TP14: TestPoint, TestPoint:TestPoint_Pad_D1.5mm, B.Cu at (116.8, 27.9)
- added TP15: TestPoint, TestPoint:TestPoint_Pad_D1.5mm, B.Cu at (114.3, 27.9)
- added TP16: TestPoint, TestPoint:TestPoint_Pad_D1.5mm, F.Cu at (82.3, 86.5)
- added U2: 74LVC1G00, Package_TO_SOT_SMD:SOT-23-5, F.Cu at (138.7, 61.3)
- added U3: CH32V003JxMx, Package_SO:SOP-8_3.9x4.9mm_P1.27mm, F.Cu at (113.4, 28.8)
- moved C6 1.02 mm to (151.4, 37.8), turned to 90 degrees
Connections:
- net Net-(C6-Pad2) renamed /S_LEFT
- net Net-(C7-Pad2) renamed /S_RIGHT
- U1 pad 12: unconnected-(U1-Pad12) -> GND
- U1 pad 13: unconnected-(U1-Pad13) -> GND
- U14 pad 1: /SAMPA18 -> GND
- U14 pad 2: /SAMPA16 -> GND
- U14 pad 30: /SAMPA17 -> GND
- U22 pad 16: /MCLK -> /~{DACWR}
- U24 pad 12: unconnected-(U24-Pad12) -> GND
- U24 pad 13: unconnected-(U24-Pad13) -> GND
- U6 pad 15: unconnected-(U6B-E-Pad15) -> +5V
Routing:
- net GND: track 194.7 -> 307.4 mm, vias 125 -> 148
- net Net-(D1-K): track 0.00 -> 54.9 mm
- net +5V: track 457.7 -> 510.2 mm, vias 33 -> 37
- net Net-(D1-A): track 0.00 -> 45.7 mm, vias 0 -> 7
- net Net-(D10-K): track 0.00 -> 38.4 mm, vias 0 -> 10
- net Net-(D13-A): track 0.00 -> 33.1 mm, vias 0 -> 9
- net Net-(D11-A): track 0.00 -> 30.4 mm, vias 0 -> 6
- net /CHX3: track 0.00 -> 27.4 mm, vias 0 -> 2
- net /CHX4: track 0.00 -> 16.0 mm
- net /MCLK: track 109.6 -> 97.4 mm, vias 4 -> 5
- net /~{DACWR}: track 0.00 -> 11.9 mm
- net Net-(C24-Pad2): track 0.00 -> 11.8 mm
- net /S_LEFT: track 15.5 -> 26.5 mm
- net /CHX5: track 0.00 -> 10.1 mm
- net /SAMPA0: track 92.7 -> 102.2 mm
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Other:
- board text added: "AB0"
- board text added: "AB1"
- board text added: "AB2"
- board text added: "AB3"
- board text added: "CH32V003 PGM"
- board text added: "DB0"
- board text added: "DB1"
- board text added: "DB2"
- board text added: "DB3"
- board text added: "DB4"
- board text added: "DB5"
- board text added: "DB6"
- board text added: "DB7"
- board text added: "GND"
- board text added: "MCLK"
- board text added: "SWDIO"
- board text added: "~{S_OE}"
- board text added: "~{S_WE}"
- board text added: "~{WRM}"
- board text added: "~{WR}"
- board text added: "~{Ф0A}"
- board text added: "~{Ф0B}"
- board text added: "~{Ф0С}"

Commit message: wip
Parts:
- added D22: LED_Small, LED_SMD:LED_0603_1608Metric, F.Cu at (70.0, 97.7)
- added D23: LED_Small, LED_SMD:LED_0603_1608Metric, F.Cu at (72.6, 97.7)
- added D24: LED_Small, LED_SMD:LED_0603_1608Metric, F.Cu at (75.2, 97.7)
- added G***: LOGO, LOGO, F.Cu at (152.4, 83.8)
- added G***: LOGO, LOGO, B.Cu at (223.9, 91.0)
- added G***: LOGO, LOGO, B.Cu at (87.1, 70.5)
- added J5: Conn_01x10, Connector_PinHeader_2.54mm:PinHeader_1x10_P2.54mm_Vertical, F.Cu at (193.0, 92.7)
- added J6: Conn_01x10, Connector_PinHeader_2.54mm:PinHeader_1x10_P2.54mm_Vertical, F.Cu at (193.0, 90.2)
- added J7: Conn_01x10, Connector_PinHeader_2.54mm:PinHeader_1x10_P2.54mm_Vertical, F.Cu at (193.0, 87.6)
- added R26: 50, Resistor_SMD:R_0805_2012Metric, F.Cu at (64.1, 71.4)
- added R27: 50, Resistor_SMD:R_0805_2012Metric, F.Cu at (130.9, 47.0)
- added R28: 720, Resistor_SMD:R_0805_2012Metric, F.Cu at (70.1, 94.1)
- added R29: 720, Resistor_SMD:R_0805_2012Metric, F.Cu at (72.6, 94.1)
- added R30: 720, Resistor_SMD:R_0805_2012Metric, F.Cu at (75.1, 94.1)
- added R31: 50, Resistor_SMD:R_0805_2012Metric, F.Cu at (78.2, 84.0)
- added R32: 50, Resistor_SMD:R_0805_2012Metric, F.Cu at (136.8, 63.9)
- added RN1: 470, Resistor_SMD:R_Array_Concave_4x0603, F.Cu at (224.2, 87.2)
- added RN2: 470, Resistor_SMD:R_Array_Concave_4x0603, F.Cu at (224.2, 92.9)
- added RN3: 470, Resistor_SMD:R_Array_Concave_4x0603, F.Cu at (186.5, 92.4)
- added RN4: 470, Resistor_SMD:R_Array_Concave_4x0603, F.Cu at (181.7, 92.3)
- added RN5: 470, Resistor_SMD:R_Array_Concave_4x0603, F.Cu at (209.0, 75.0)
- added RN6: 470, Resistor_SMD:R_Array_Concave_4x0603, F.Cu at (196.5, 75.1)
- added U20: Pico, MCU_RaspberryPi_and_Boards:RPi_Pico_SMD_TH, B.Cu at (204.5, 71.8)
- added U25: 74AUP1G08, Package_TO_SOT_SMD:SOT-353_SC-70-5, F.Cu at (94.2, 32.2)
- added U27: 74LVC1G332, Package_TO_SOT_SMD:SOT-23-6, F.Cu at (97.3, 32.1)
- U2: footprint Package_TO_SOT_SMD:SOT-23-5 -> Package_TO_SOT_SMD:SOT-353_SC-70-5
- moved R20 14.7 mm to (110.7, 27.8), turned to 90 degrees
- moved C22 2.67 mm to (124.7, 29.6)
- moved C23 2.67 mm to (123.4, 35.3)
- moved C24 2.67 mm to (125.1, 32.8)
- moved C7 2.67 mm to (131.0, 29.8)
- moved D21 2.67 mm to (119.6, 33.7)
- moved J4 2.67 mm to (142.4, 29.8)
- moved R16 2.67 mm to (134.6, 35.2)
- moved R17 2.67 mm to (115.8, 32.8)
- moved R22 2.67 mm to (130.6, 35.1)
- moved R23 2.67 mm to (125.7, 26.9)
- moved R24 2.67 mm to (122.6, 28.1)
- moved R25 2.67 mm to (122.6, 31.9)
- moved TP13 2.67 mm to (114.4, 27.9)
- moved TP14 2.67 mm to (119.5, 27.9)
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Connections:
- J3 pad 3: unconnected-(J3-Pin_3-Pad3) -> /~{LOOPEN_B}
- U11 pad 11: /PITCHx256_B -> /Px256_B_GATED
- U11 pad 13: /PITCHx256_B -> /Px256_B_GATED
- U11 pad 9: unconnected-(U11-~{RCO}-Pad9) -> /~{RCO_B}
- U26 pad 4: /~{DACA}/DACB -> Net-(R26-Pad2)
- X1 pad 3: /MCLK -> Net-(X1-OUT)
Routing:
- net /~{LOOPEN_B}: track 0.00 -> 122.2 mm, vias 0 -> 1
- net GND: track 307.4 -> 421.9 mm, vias 148 -> 192
- net /PI_5V: track 0.00 -> 58.2 mm, vias 0 -> 1
- net /PI_DB7: track 0.00 -> 37.1 mm
- net /PI_DB6: track 0.00 -> 36.0 mm
- net Net-(RN5-R4.2): track 0.00 -> 35.6 mm, vias 0 -> 1
- net Net-(RN5-R3.2): track 0.00 -> 32.4 mm, vias 0 -> 1
- net /PI_AB0: track 0.00 -> 30.2 mm, vias 0 -> 2
- net /PI_AB1: track 0.00 -> 29.6 mm, vias 0 -> 2
- net /PI_AB2: track 0.00 -> 28.6 mm, vias 0 -> 2
- net /PI_DB5: track 0.00 -> 28.2 mm, vias 0 -> 2
- net /~{PI_SRAM_OE}: track 0.00 -> 28.1 mm, vias 0 -> 2
- net /PI_AB3: track 0.00 -> 27.5 mm, vias 0 -> 2
- net /~{PI_SRAM_WE}: track 0.00 -> 27.3 mm, vias 0 -> 2
- net /PI_DB4: track 0.00 -> 27.1 mm, vias 0 -> 2
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- added copper zone on B.Cu, net /PI_GND
- added copper zone on F.Cu, net /PI_GND
Other:
- board size 99.1 x 74.9 mm -> 168.9 x 76.2 mm
- board text added: "2024"
- board text added: "https://github.com/svofski/lepetomane-ringard"
- board text added: "review SOT-353 and SOT-363 single-gate packages!"
- board text added: "~{ЛУПЕНЬ {dblquote}Б{dblquote}}"

Commit message: before separation
Connections:
- net Net-(RN1-R1.1) renamed /PI_GPIO0
- net Net-(RN1-R2.1) renamed /PI_GPIO1
- net Net-(RN1-R3.1) renamed /PI_GPIO2
- net Net-(RN1-R4.1) renamed /PI_GPIO3
- net Net-(RN2-R1.1) renamed /PI_GPIO4
- net Net-(RN2-R2.1) renamed /PI_GPIO5
- net Net-(RN2-R3.1) renamed /PI_GPIO6
- net Net-(RN2-R4.1) renamed /PI_GPIO7
- net Net-(RN3-R1.1) renamed /PI_GPIO8
- net Net-(RN3-R2.1) renamed /PI_GPIO9
- net Net-(RN3-R3.1) renamed /PI_GPIO10
- net Net-(RN3-R4.1) renamed /PI_GPIO11
- net Net-(RN4-R1.1) renamed /PI_GPIO12
- net Net-(RN4-R2.1) renamed /PI_GPIO13
- net Net-(RN4-R3.1) renamed /PI_GPIO14
- net Net-(RN4-R4.1) renamed /PI_GPIO15
- net Net-(RN5-R1.2) renamed /PI_GPIO19
- net Net-(RN5-R2.2) renamed /PI_GPIO18
- net Net-(RN5-R3.2) renamed /PI_GPIO17
- net Net-(RN5-R4.2) renamed /PI_GPIO16
- net Net-(RN6-R1.2) renamed /PI_GPIO26
- net Net-(RN6-R2.2) renamed /PI_GPIO22
- net Net-(RN6-R3.2) renamed /PI_GPIO21
- net Net-(RN6-R4.2) renamed /PI_GPIO20
- U20 pad 36: unconnected-(U20-3V3-Pad36) -> /PI_3V3
Other:
- outline, holes or cut-outs redrawn

Commit message: as ordered
Parts:
- removed the G*** at (223.9, 91.0)
- removed J5, J6, J7: Conn_01x10, Connector_PinHeader_2.54mm:PinHeader_1x10_P2.54mm_Vertical
- removed RN1, RN2, RN3, RN4, RN5, RN6: 470, Resistor_SMD:R_Array_Concave_4x0603
- removed U20: Pico, MCU_RaspberryPi_and_Boards:RPi_Pico_SMD_TH
- added C25: 220uF/16V, Capacitor_Tantalum_SMD:CP_EIA-7343-31_Kemet-D, F.Cu at (72.5, 36.8)
- added C26: 220uF/16V, Capacitor_Tantalum_SMD:CP_EIA-7343-31_Kemet-D, F.Cu at (148.3, 72.8)
- added C27: 220uF/16V, Capacitor_Tantalum_SMD:CP_EIA-7343-31_Kemet-D, F.Cu at (120.9, 93.7)
- added C28: 10uF, Capacitor_SMD:C_0805_2012Metric, F.Cu at (139.3, 43.3)
- added C29: 10uF, Capacitor_SMD:C_0805_2012Metric, F.Cu at (121.7, 78.3)
- added C30: 10uF, Capacitor_SMD:C_0805_2012Metric, F.Cu at (112.0, 54.3)
- added C31: 10uF, Capacitor_SMD:C_0805_2012Metric, F.Cu at (78.4, 74.0)
- added C32: 100nF, Capacitor_SMD:C_0402_1005Metric, F.Cu at (75.1, 90.4)
- added TP17: TestPoint, TestPoint:TestPoint_Pad_D1.5mm, F.Cu at (137.5, 95.5)
- added TP18: TestPoint, TestPoint:TestPoint_Pad_D1.5mm, F.Cu at (74.4, 30.9)
- C1, C10, C11, C2, C22, C3, C8, C9: footprint Capacitor_SMD:C_0603_1608Metric -> Capacitor_SMD:C_0402_1005Metric
- C24: footprint Capacitor_SMD:C_0603_1608Metric -> Capacitor_SMD:C_0805_2012Metric
- U6: value 74LS139 -> 74HC139
- moved TP1 9.67 mm to (153.7, 77.3)
- moved TP4 7.62 mm to (153.8, 74.2)
- moved TP5 7.62 mm to (153.9, 70.2)
- moved C22 3.95 mm to (120.8, 29.5)
- moved R17 1.70 mm to (114.1, 33.1)
- moved G*** 1.23 mm to (151.2, 84.0)
- moved TP8 1.22 mm to (65.8, 67.5)
- moved C24 0.97 mm to (125.1, 31.8)
- moved R26 0.82 mm to (64.1, 70.5)
- moved C8 0.77 mm to (104.7, 72.1), turned to 180 degrees
- moved D22 0.25 mm to (70.0, 97.4)
- moved D23 0.25 mm to (72.6, 97.4)
- moved D24 0.25 mm to (75.2, 97.4)
Routing:
- net GND: track 421.9 -> 544.4 mm, vias 192 -> 217
- net +5V: track 528.6 -> 598.1 mm, vias 38 -> 41
- net /PI_5V: track 58.2 -> 0.00 mm, vias 1 -> 0
- net /PI_DB7: track 37.1 -> 0.00 mm
- net /PI_DB6: track 36.0 -> 0.00 mm
- net /PI_GPIO16: track 35.6 -> 0.00 mm, vias 1 -> 0
- net /PI_GPIO17: track 32.4 -> 0.00 mm, vias 1 -> 0
- net /PI_AB0: track 30.2 -> 0.00 mm, vias 2 -> 0
- net /PI_AB1: track 29.6 -> 0.00 mm, vias 2 -> 0
- net /PI_AB2: track 28.6 -> 0.00 mm, vias 2 -> 0
- net /PI_DB5: track 28.2 -> 0.00 mm, vias 2 -> 0
- net /~{PI_SRAM_OE}: track 28.1 -> 0.00 mm, vias 2 -> 0
- net /PI_AB3: track 27.5 -> 0.00 mm, vias 2 -> 0
- net /~{PI_SRAM_WE}: track 27.3 -> 0.00 mm, vias 2 -> 0
- net /PI_DB4: track 27.1 -> 0.00 mm, vias 2 -> 0
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- removed copper zone on B.Cu, net /PI_GND
- removed copper zone on F.Cu, net /PI_GND
Other:
- board size 168.9 x 76.2 mm -> 99.1 x 74.9 mm
- board text added: "JLCJLCJLCJLC"
- board text added: "LEFT"
- board text added: "MV"
- board text added: "PP"
- board text added: "Q0"
- board text added: "Q1"
- board text added: "Q2"
- board text added: "Q3"
- board text added: "Q4"
- board text added: "Q5"
- board text added: "Q6"
- board text added: "RIGHT"
- board text added: "TMR"
- board text added: "VU"
- board text added: "X"
- board text added: "~{ЛУПЕНЬ{dblquote}Б{dblquote}}"
- board text removed: "review SOT-353 and SOT-363 single-gate packages!"
- board text removed: "~{ЛУПЕНЬ {dblquote}Б{dblquote}}"
