File: kicad/neopeto/neopeto.kicad_sch (KiCad schematic)
At the start: 144 parts, among them J1 Conn_01x10_Pin, J2 Conn_01x10_Pin, J3 Conn_01x10_Pin, J4 PJ-307, U1 74HC00, U10 74HC590, U11 74HC590, U12 74HC590, U13 74HC245, U14 K6X4008C1F, U15 74HC245, U16 74HC245, U17 LM358LV, U18 LM358LV, U19 LM358LV, U2 74LVC1G00, U21 TLC7258C, U22 TLC7258C, U23 74HC4017, U24 74HC86, U25 74AUP1G08, U26 74LVC1G332, U27 74LVC1G332, U3 CH32V003JxMx, U4 82C55A_PLCC, U5 82C54_PLCC, U6 74HC139, U7 74HC245, U8 74HC245, U9 74HC245, X1 ECS-2520MV-12MHZ

Commit message: schematic update with scopes
Parts:
- R27, R32: now not fitted
- X1: value ECS-2520MV-12MHZ -> ECS-2520MV-8MHZ
Other:
- note added: "1.33 MHz"
- note added: "CHOPPER MODE"
- note added: "SAMPLE ADDR MSB ~{WRMODE}=1 ~{SRAM_OE}=0"
- note added: "WRITE MODE"
- note added: "~{WRMODE}=0 ~{SRAM_OE}=1 ~{SRAM_WE} \ -> SRAM[PB,PA] = PC"
- note removed: "CHOPPER MODE SAMPLE ADDR MSB ~{WRMODE}=1 ~{SRAM_OE}=0"
- note removed: "WRITE MODE ~{WRMODE}=0 ~{SRAM_OE}=1 ~{SRAM_WE} \ -> SRAM[PB,PA] = PC"
