File: kicad/neopeto/neopeto.kicad_sch (KiCad schematic)
At the start: 144 parts, among them J1 Conn_01x10_Pin, J2 Conn_01x10_Pin, J3 Conn_01x10_Pin, J4 PJ-307, U1 74HC00, U10 74HC590, U11 74HC590, U12 74HC590, U13 74HC245, U14 K6X4008C1F, U15 74HC245, U16 74HC245, U17 LM358LV, U18 LM358LV, U19 LM358LV, U2 74LVC1G00, U21 TLC7258C, U22 TLC7258C, U23 74HC4017, U24 74HC86, U25 74AUP1G08, U26 74LVC1G332, U27 74LVC1G332, U3 CH32V003JxMx, U4 82C55A_PLCC, U5 82C54_PLCC, U6 74HC139, U7 74HC245, U8 74HC245, U9 74HC245, X1 ECS-2520MV-8MHZ

Commit message: test notes in the schematic + debug monitor
debug monitor provides some basic commands to test the circuit
Other:
- note added: "TEST: CTR0 div=100 PITCHx256_A = 80kHz U10.~{RCO} = 312.5Hz"
Changed lines of the file:
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@@
 		)
 	)
-	(polyline
-		(pts
-			(xy 65.405 52.705) (xy 65.405 19.685)
-		)
-		(stroke
-			(width 0)
-			(type default)
-		)
-	)
 	(wire
 		(pts
@@
 		)
 	)
+	(polyline
+		(pts
+			(xy 65.405 29.21) (xy 65.405 38.735)
+		)
+		(stroke
+			(width 0)
+			(type default)
+		)
+	)
 	(wire
 		(pts
@@
 		)
 	)
+	(polyline
+		(pts
+			(xy 55.88 29.21) (xy 65.405 29.21)
+		)
+		(stroke
+			(width 0)
+			(type default)
+		)
+	)
 	(wire
 		(pts
@@
 		)
 	)
+	(polyline
+		(pts
+			(xy 236.22 52.705) (xy 236.22 59.055)
+		)
+		(stroke
+			(width 0)
+			(type default)
+		)
+	)
 	(wire
 		(pts
@@
 		)
 	)
-	(polyline
-		(pts
-			(xy 65.405 8.89) (xy 65.405 19.685)
-		)
-		(stroke
-			(width 0)
-			(type default)
-		)
-	)
 	(wire
 		(pts
@@
 		)
 	)
+	(polyline
+		(pts
+			(xy 190.5 59.055) (xy 236.22 59.055)
+		)
+		(stroke
+			(width 0)
+			(type default)
+		)
+	)
 	(wire
 		(pts
@@
 		)
 	)
-	(polyline
-		(pts
-			(xy 125.73 8.89) (xy 172.085 8.89)
-		)
-		(stroke
-			(width 0)
-			(type default)
-		)
-	)
 	(wire
 		(pts
@@
 		)
 	)
-	(polyline
-		(pts
-			(xy 125.73 36.83) (xy 125.73 8.89)
-		)
-		(stroke
-			(width 0)
-			(type default)
-		)
-	)
 	(wire
 		(pts
@@
 	)
 	(image
-		(at 55.88 -3.175)
+		(at 57.15 20.955)
+		(scale 0.389478)
 		(data "iVBORw0KGgoAAAANSUhEUgAAAeAAAAEQCAIAAADnJDDbAAAgAElEQVR4nO19LZjiyPf1+b9PxBWI"
 			"Ei0iWkS0QIyIaIEYgRiBGIEYgRiB+AnEihYrECMQKxAjECsQKxArECsQKxAjIlYgRiBGIEYgRkS0"
@@
 	)
 	(image
-		(at 151.765 30.48)
+		(at 153.035 36.195)
 		(scale 0.25)
 		(data "iVBORw0KGgoAAAANSUhEUgAAAf0AAAGBCAIAAADjTv9lAAAA0mVYSWZJSSoACAAAAAoAAAEEAAEA"
@@
 		)
 	)
+	(text "TEST: CTR0 div=100\nPITCHx256_A = 80kHz\nU10.~{RCO} = 312.5Hz"
+		(exclude_from_sim no)
+		(at 190.5 55.88 0)
+		(effects
+			(font
+				(size 1.27 1.27)
+			)
+			(justify left)
+		)
+	)
 	(text "SAMPLE ADDR MSB\n~{WRMODE}=1\n~{SRAM_OE}=0"
 		(exclude_from_sim no)
@@
 	(text "1.33 MHz"
 		(exclude_from_sim no)
-		(at 60.325 22.225 0)
+		(at 60.325 27.94 0)
 		(effects
 			(font
